File: eagle sch + brd/numitron_tube_clock.sch (EAGLE design)
At the start: 39 parts, among them IC1 MAX7219CNG, IC2 MEGA8-AI, IC4 DS1307, Q1 12 MHz, Q2 32kHz, X2 MINI-USB-UX60-MB-5S8

Commit message: added power button and generated board
added power button and generated board
Parts:
- added S2: SWITCH-MOMENTARY-2SMD, SparkFun-Electromechanical:SWITCH-MOMENTARY-2SMD
- IC1: value MAX7219CNG -> MAX7219CWG; device maxim:MAX7219CNG -> max7219:MAX7219CWG
- IC4: value DS1307 -> DS1307Z; device ds1307_pcf8583:DS1307 -> ds1307_pcf8583:DS1307Z
Connections:
- net +3V3: now also S2.1
- net GND: now also S2.2
Changed lines of the file:
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@@
 </classes>
 <parts>
-<part name="IC1" library="maxim" deviceset="MAX7219CNG" device=""/>
+<part name="IC1" library="max7219" deviceset="MAX7219CWG" device=""/>
 <part name="IC2" library="atmel" deviceset="MEGA8" device="-AI"/>
 <part name="Q1" library="crystal" deviceset="CRYSTAL" device="HC49U-V" value="12 MHz"/>
@@
 <part name="SUPPLY21" library="supply2" deviceset="GND" device=""/>
 <part name="SUPPLY22" library="supply2" deviceset="GND" device=""/>
-<part name="IC4" library="ds1307_pcf8583" deviceset="DS1307" device=""/>
+<part name="IC4" library="ds1307_pcf8583" deviceset="DS1307" device="Z" value="DS1307Z"/>
 <part name="Q2" library="crystal" deviceset="CRYSTAL" device="HC49U-V" value="32kHz"/>
 <part name="P+7" library="supply1" deviceset="+5V" device=""/>
@@
 <part name="P+6" library="supply1" deviceset="+5V" device=""/>
 <part name="SUPPLY17" library="supply2" deviceset="GND" device=""/>
+<part name="+3V7" library="supply1" deviceset="+3V3" device=""/>
+<part name="+3V8" library="supply1" deviceset="+3V3" device=""/>
+<part name="SUPPLY23" library="supply2" deviceset="GND" device=""/>
+<part name="S2" library="SparkFun-Electromechanical" deviceset="SWITCH-MOMENTARY-2" device="SMD"/>
 </parts>
 <sheets>
@@
 <instance part="P+6" gate="1" x="186.87" y="5.52"/>
 <instance part="SUPPLY17" gate="GND" x="187.18" y="-15.51"/>
+<instance part="+3V7" gate="G$1" x="-18.91" y="-35.24"/>
+<instance part="+3V8" gate="G$1" x="-7.91" y="-36.69" rot="R90"/>
+<instance part="SUPPLY23" gate="GND" x="7.75" y="-36.69" rot="R90"/>
+<instance part="S2" gate="G$1" x="-0.11" y="-36.69"/>
 </instances>
 <busses>
@@
 <junction x="-19.2" y="-41.22"/>
 </segment>
+<segment>
+<pinref part="S2" gate="G$1" pin="2"/>
+<pinref part="SUPPLY23" gate="GND" pin="GND"/>
+<wire x1="4.97" y1="-36.69" x2="5.21" y2="-36.69" width="0.1524" layer="91"/>
+</segment>
 </net>
 <net name="N$53" class="0">
@@
 <wire x1="-18.91" y1="-37.78" x2="-18.91" y2="-37.72" width="0.1524" layer="91"/>
 <junction x="-18.91" y="-37.78"/>
-</segment>
-</net>
+<pinref part="+3V7" gate="G$1" pin="+3V3"/>
+</segment>
+<segment>
+<wire x1="-5.43" y1="-36.69" x2="-5.37" y2="-36.69" width="0.1524" layer="91"/>
+<pinref part="+3V8" gate="G$1" pin="+3V3"/>
+<wire x1="-5.37" y1="-36.69" x2="-5.19" y2="-36.69" width="0.1524" layer="91"/>
+<junction x="-5.37" y="-36.69"/>
+<pinref part="S2" gate="G$1" pin="1"/>
+<wire x1="-5.19" y1="-36.69" x2="-5.06" y2="-36.69" width="0.1524" layer="91"/>
+<junction x="-5.19" y="-36.69"/>
+</segment>
+</net>
