File: eagle sch + brd/numi_clock.sch (EAGLE design)
At the start: 37 parts, among them IC1 MEGA8-AI, IC2 LM75, Q1 12MHz, Y1 32.768kHz

Commit message: layout adjustments
layout adjustments
Parts:
- removed C6, C7, C8: 100nF, rcl:C-EUC0805
- removed D3, D4: red, SparkFun-LED:LED1206
- removed R9: 10k, rcl:R-EU_R0805
- removed SV1: SPI, con-lstb:MA03-2
- removed SV7: dig0, con-lstb:MA09-1
- added SV3: (no value), con-lstb:MA08-1
Connections:
- removed net LED: D4.A, IC1.ADC7
- removed net MISO: IC1.PB4(MISO), SV1.1
- net +5V: no longer C6.2, C7.2, C8.2, D3.A, IC1.AVCC, R9.1, SV1.2
- net A: now also SV3.8; no longer SV7.5
- net B: now also SV3.7, U$1.SEGF; no longer SV7.3, U$1.SEGB
- net C: now also SV3.6, U$1.SEGB; no longer SV7.4, U$1.SEGC
- net D: now also SV3.5, U$1.SEGG; no longer SV7.8, U$1.SEGD
- net DIG0: no longer R9.2, SV7.1
- net DIG1: now also U$1.DIG2; no longer U$1.DIG1
- net DIG2: now also U$1.DIG3; no longer U$1.DIG2
- net DIG3: now also U$1.DIG1; no longer U$1.DIG3
- net DP: now also SV3.1, U$1.SEGD; no longer SV7.2, U$1.SEGDP
- net E: now also SV3.4, U$1.SEGC; no longer SV7.9, U$1.SEGE
- net F: now also SV3.3, U$1.SEGE; no longer SV7.6, U$1.SEGF
- net FUNC: now also IC1.ADC7; no longer IC1.ADC6
- net G: now also SV3.2, U$1.SEGDP; no longer SV7.7, U$1.SEGG
- net GND: no longer C6.1, C7.1, C8.1, D3.C, D4.C, SV1.6
- net HC: now also IC1.PB1(OC1A); no longer IC1.PC0(ADC0)
- net HOUR: now also IC1.PC3(ADC3); no longer IC1.PC2(ADC2)
- net MINUTE: now also IC1.PC2(ADC2); no longer IC1.PC3(ADC3)
- net MOSI: no longer SV1.4
- net N$10: now also IC1.PD7(AIN1); no longer IC1.PD3(INT1)
- net RESET: no longer SV1.5
- net SCK: no longer SV1.3
Other:
- moved on the sheet: SV8

Commit message: routed all tracks
routed all tracks
Parts:
- added D3: (no value), sym:LED
Connections:
- new net LED: D3.+, IC1.ADC6
- net GND: now also D3.-
Changed lines of the file:
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@@
 <part name="SV8" library="con-lstb" deviceset="MA04-1" device="" value="conn digits"/>
 <part name="SV3" library="con-lstb" deviceset="MA08-1" device=""/>
+<part name="SUPPLY8" library="supply2" deviceset="GND" device=""/>
+<part name="D3" library="sym" deviceset="LED" device=""/>
 </parts>
 <sheets>
@@
 <instance part="SV8" gate="1" x="-142.24" y="43.18" rot="MR180"/>
 <instance part="SV3" gate="1" x="7.62" y="43.18"/>
+<instance part="SUPPLY8" gate="GND" x="116.84" y="50.8"/>
+<instance part="D3" gate="G$1" x="114.3" y="63.5"/>
 </instances>
 <busses>
@@
 <pinref part="SUPPLY25" gate="GND" pin="GND"/>
 <wire x1="86.36" y1="96.52" x2="83.82" y2="96.52" width="0.1524" layer="91"/>
+</segment>
+<segment>
+<pinref part="SUPPLY8" gate="GND" pin="GND"/>
+<pinref part="D3" gate="G$1" pin="-"/>
 </segment>
 </net>
@@
 </segment>
 </net>
+<net name="LED" class="0">
+<segment>
+<pinref part="IC1" gate="G$1" pin="ADC6"/>
+<wire x1="-78.74" y1="129.54" x2="-76.2" y2="129.54" width="0.1524" layer="91"/>
+<label x="-76.2" y="129.54" size="1.778" layer="95"/>
+</segment>
+<segment>
+<wire x1="116.84" y1="63.5" x2="116.84" y2="66.04" width="0.1524" layer="91"/>
+<label x="116.84" y="66.04" size="1.778" layer="95"/>
+<pinref part="D3" gate="G$1" pin="+"/>
+</segment>
+</net>
