File: hardware/numi_clock.brd (EAGLE design)
At the start: 70.8 x 29.5 mm, 31 parts, among them IC1 MEGA8-AI, IC2 LM75, Q1 12MHz, Y1 32.768kHz

Commit message: first software upload
restructured directory tree, commit barebone max7219 example
Parts:
- moved S2 4.92 mm to (77.0, 9.37), turned to 0 degrees
- moved S1 3.53 mm to (68.1, 9.37), turned to 0 degrees
- moved S3 3.29 mm to (32.8, 9.37)
- moved Y1 0.28 mm to (43.9, 13.8)
Routing:
- net FUNC: track 93.2 -> 45.6 mm
- net +5V: track 227.3 -> 209.2 mm
- net HOUR: track 22.0 -> 20.2 mm
- net MINUTE: track 28.0 -> 26.9 mm
- net GND: track 80.4 -> 81.3 mm
- net N$4: track 8.73 -> 8.21 mm
Changed lines of the file:
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@@
 <?xml version="1.0" encoding="utf-8"?>
 <!DOCTYPE eagle SYSTEM "eagle.dtd">
-<eagle version="7.4.0">
+<eagle version="7.3.0">
 <drawing>
 <settings>
@@
 <dimension x1="15.125" y1="37.5" x2="15.125" y2="8" x3="11.5" y3="22.75" textsize="1.778" layer="20"/>
 <dimension x1="15.125" y1="37.5" x2="85.875" y2="37.5" x3="50.5" y3="41.375" textsize="1.778" layer="20"/>
+<dimension x1="15.125" y1="8" x2="50.5" y2="8.125" x3="32.840871875" y3="0.03300625" textsize="1.778" layer="20"/>
+<dimension x1="15.125" y1="8" x2="32.875" y2="8" x3="24" y3="5.375" textsize="1.778" layer="20"/>
+<dimension x1="85.875" y1="8" x2="77" y2="8" x3="81.4375" y3="5.25" textsize="1.778" layer="20"/>
+<dimension x1="85.875" y1="8" x2="68.125" y2="7.875" x3="77.059840625" y3="-0.560321875" textsize="1.778" layer="20"/>
 </plain>
 <attributes>
@@
 <element name="R4" library="rcl" package="R0805" value="68" x="35" y="29.5" rot="MR270"/>
 <element name="R8" library="rcl" package="R0805" value="10k" x="56.875" y="21.5" rot="MR0"/>
-<element name="S1" library="SparkFun-Electromechanical" package="TACTILE_SWITCH-SMD-RIGHT-ANGLE" value="SWITCH-MOMENTARY-2TACTILE-SWITCH-SMD-RIGHT-ANGLE" x="68.425" y="12.88" rot="MR180">
-<attribute name="PROD_ID" value="COMP-12265" x="68.425" y="12.88" size="1.778" layer="28" rot="MR180" display="off"/>
-</element>
-<element name="S2" library="SparkFun-Electromechanical" package="TACTILE_SWITCH-SMD-RIGHT-ANGLE" value="SWITCH-MOMENTARY-2TACTILE-SWITCH-SMD-RIGHT-ANGLE" x="77.54" y="14.255" rot="MR180">
-<attribute name="PROD_ID" value="COMP-12265" x="77.54" y="14.255" size="1.778" layer="28" rot="MR180" display="off"/>
+<element name="S1" library="SparkFun-Electromechanical" package="TACTILE_SWITCH-SMD-RIGHT-ANGLE" value="SWITCH-MOMENTARY-2TACTILE-SWITCH-SMD-RIGHT-ANGLE" x="68.075" y="9.37" rot="MR0">
+<attribute name="PROD_ID" value="COMP-12265" x="68.075" y="9.37" size="1.778" layer="28" rot="MR0" display="off"/>
+</element>
+<element name="S2" library="SparkFun-Electromechanical" package="TACTILE_SWITCH-SMD-RIGHT-ANGLE" value="SWITCH-MOMENTARY-2TACTILE-SWITCH-SMD-RIGHT-ANGLE" x="76.96" y="9.37" rot="MR0">
+<attribute name="PROD_ID" value="COMP-12265" x="76.96" y="9.37" size="1.778" layer="28" rot="MR0" display="off"/>
 </element>
 <element name="SV2" library="con-lstb" package="MA03-1" value="HC-SR505" x="50.16" y="34.75">
@@
 <element name="U$1" library="max7219" package="SO24L" value="MAX7219CWG" x="71.53" y="25.8" rot="MR0"/>
 <element name="U$2" library="SparkFun-FreqCtrl" package="SO08" value="DS1307SO8" x="50.25" y="14.375" rot="MR90"/>
-<element name="Y1" library="SparkFun-FreqCtrl" package="TC26H" value="32.768kHz" x="43.625" y="13.875" rot="R90">
-<attribute name="PROD_ID" value="XTAL-10112" x="43.625" y="13.875" size="1.778" layer="27" rot="R90" display="off"/>
-</element>
-<element name="S3" library="SparkFun-Electromechanical" package="TACTILE_SWITCH-SMD-RIGHT-ANGLE" value="SWITCH-MOMENTARY-2TACTILE-SWITCH-SMD-RIGHT-ANGLE" x="33.305" y="12.62" rot="MR0">
-<attribute name="PROD_ID" value="COMP-12265" x="33.305" y="12.62" size="1.778" layer="28" rot="MR0" display="off"/>
+<element name="Y1" library="SparkFun-FreqCtrl" package="TC26H" value="32.768kHz" x="43.875" y="13.75" rot="R90">
+<attribute name="PROD_ID" value="XTAL-10112" x="43.875" y="13.75" size="1.778" layer="27" rot="R90" display="off"/>
+</element>
+<element name="S3" library="SparkFun-Electromechanical" package="TACTILE_SWITCH-SMD-RIGHT-ANGLE" value="SWITCH-MOMENTARY-2TACTILE-SWITCH-SMD-RIGHT-ANGLE" x="32.805" y="9.37" rot="MR0">
+<attribute name="PROD_ID" value="COMP-12265" x="32.805" y="9.37" size="1.778" layer="28" rot="MR0" display="off"/>
 </element>
 <element name="BAT2" library="SparkFun" package="BATTCOM_20MM_PTH" value="cr2032" x="26.075" y="33.815" rot="R270"/>
@@
 <contactref element="C10" pad="1"/>
 <wire x1="68.355" y1="20.7708" x2="68.375" y2="20.7908" width="0.4064" layer="16"/>
-<wire x1="31.355" y1="12.62" x2="31.225" y2="12.75" width="0.5" layer="16"/>
+<wire x1="30.855" y1="9.37" x2="31.225" y2="12.75" width="0.5" layer="16"/>
 <polygon width="0.254" layer="16" isolate="0.4064">
 <vertex x="15.25" y="37.375"/>
@@
 <wire x1="74.875" y1="15.625" x2="75.75" y2="15.625" width="0.4064" layer="16"/>
 <wire x1="75.75" y1="15.625" x2="75.875" y2="15.75" width="0.4064" layer="16"/>
-<wire x1="79.49" y1="14.255" x2="79.49" y2="16.51" width="0.4064" layer="16"/>
+<wire x1="75.01" y1="9.37" x2="79.49" y2="16.51" width="0" layer="19" extent="1-16"/>
 <wire x1="79.49" y1="16.51" x2="78.625" y2="17.375" width="0.4064" layer="16"/>
 <wire x1="42.1" y1="22.675" x2="42.925" y2="22.175" width="0.4064" layer="16"/>
@@
 <wire x1="37.5" y1="22.375" x2="39.825" y2="22.375" width="0.4064" layer="16"/>
 <wire x1="39.825" y1="22.375" x2="40" y2="22.55" width="0.4064" layer="16"/>
+<wire x1="66.125" y1="9.37" x2="73.5" y2="15.875" width="0" layer="19" extent="16-16"/>
+<wire x1="59.7" y1="18.84" x2="56.11" y2="26.36" width="0" layer="19" extent="16-16"/>
 </signal>
 <signal name="N$1">
@@
 <wire x1="81.75" y1="26.125" x2="81.75" y2="11.75" width="0.45" layer="16"/>
 <wire x1="81.75" y1="11.75" x2="81" y2="11" width="0.45" layer="16"/>
-<wire x1="81" y1="11" x2="62.875" y2="11" width="0.45" layer="16"/>
+<wire x1="81" y1="11" x2="62.875" y2="11" width="0" layer="19" extent="1-16"/>
 <wire x1="62.875" y1="11" x2="55.875" y2="11" width="0.45" layer="16"/>
 <wire x1="55.875" y1="11" x2="37.75" y2="11" width="0.45" layer="16"/>
@@
 <contactref element="C9" pad="2"/>
 <contactref element="Y1" pad="1"/>
-<wire x1="43.625" y1="12.605" x2="45.01" y2="12.47" width="0.5" layer="16"/>
+<wire x1="43.875" y1="12.48" x2="45.01" y2="12.47" width="0.5" layer="16"/>
 <wire x1="45.01" y1="12.47" x2="47.6338" y2="12.47" width="0.5" layer="16"/>
 <wire x1="40.825" y1="12.75" x2="44.25" y2="12.75" width="0.5" layer="16"/>
 <wire x1="44.25" y1="12.75" x2="44.52" y2="12.48" width="0.5" layer="16"/>
-<wire x1="44.52" y1="12.48" x2="43.625" y2="12.605" width="0.5" layer="16"/>
+<wire x1="44.52" y1="12.48" x2="43.875" y2="12.48" width="0.5" layer="16"/>
 </signal>
 <signal name="N$7">
@@
 <contactref element="S1" pad="1"/>
 <contactref element="IC1" pad="26"/>
-<wire x1="66.475" y1="12.88" x2="66.475" y2="14.65" width="0.4064" layer="16"/>
+<wire x1="70.025" y1="9.37" x2="66.475" y2="14.65" width="0" layer="19" extent="1-16"/>
 <wire x1="66.475" y1="14.65" x2="64.875" y2="16.25" width="0.4064" layer="16"/>
 <wire x1="64.875" y1="16.25" x2="64.875" y2="17.5" width="0.4064" layer="16"/>
@@
 <via x="63" y="25.875" extent="1-16" drill="0.8"/>
 <wire x1="63" y1="25.875" x2="80.375" y2="25.875" width="0.4064" layer="16"/>
-<wire x1="35.255" y1="12.62" x2="35.255" y2="11.745" width="0.45" layer="16"/>
-<wire x1="35.255" y1="11.745" x2="36.875" y2="10.125" width="0.45" layer="16"/>
-<wire x1="36.875" y1="10.125" x2="81.25" y2="10.125" width="0.45" layer="16"/>
+<wire x1="34.755" y1="9.37" x2="35.255" y2="11.745" width="0" layer="19" extent="1-16"/>
+<wire x1="35.255" y1="11.745" x2="36.875" y2="10.125" width="0" layer="19" extent="1-16"/>
+<wire x1="36.875" y1="10.125" x2="81.25" y2="10.125" width="0" layer="19" extent="1-16"/>
 <wire x1="81.25" y1="10.125" x2="83" y2="11.625" width="0.45" layer="16"/>
 <wire x1="83" y1="11.625" x2="83" y2="25.875" width="0.45" layer="16"/>
@@
 <contactref element="S2" pad="1"/>
 <contactref element="IC1" pad="25"/>
-<wire x1="75.59" y1="14.255" x2="74.505" y2="14.255" width="0.5" layer="16"/>
+<wire x1="78.91" y1="9.37" x2="74.505" y2="14.255" width="0" layer="19" extent="1-16"/>
 <wire x1="74.505" y1="14.255" x2="74.5" y2="14.25" width="0.5" layer="16"/>
 <wire x1="74.5" y1="14.25" x2="74.375" y2="14.25" width="0.5" layer="16"/>
@@
 <contactref element="Y1" pad="2"/>
 <wire x1="40.95" y1="15.125" x2="42.595" y2="15.02" width="0.5" layer="16"/>
-<wire x1="42.595" y1="15.02" x2="43.625" y2="15.145" width="0.5" layer="16"/>
+<wire x1="42.595" y1="15.02" x2="43.875" y2="15.02" width="0.5" layer="16"/>
 <wire x1="47.6338" y1="13.74" x2="47.6238" y2="13.75" width="0.5" layer="16"/>
 <wire x1="47.6238" y1="13.75" x2="45.125" y2="13.75" width="0.5" layer="16"/>
 <wire x1="45.125" y1="13.75" x2="43.73" y2="15.145" width="0.5" layer="16"/>
-<wire x1="43.73" y1="15.145" x2="43.625" y2="15.145" width="0.5" layer="16"/>
+<wire x1="43.73" y1="15.145" x2="43.875" y2="15.02" width="0.5" layer="16"/>
 </signal>
 <signal name="AVCC">

Commit message: layout adjustments
layout adjustments
Parts:
- moved R11 18.1 mm to (80.6, 27.6), turned to 270 degrees
- moved C4 8.93 mm to (47.2, 35.1), turned to 270 degrees
- moved D3 3.54 mm to (59.9, 27.4), turned to 270 degrees
- moved SV2 2.64 mm to (52.8, 35.0)
- moved R8 0.25 mm to (56.9, 21.2)
Routing:
- net HOUR: track 20.2 -> 28.7 mm
- net GND: track 81.3 -> 89.6 mm, vias 8 -> 6
- net MINUTE: track 26.9 -> 34.9 mm
- net +5V: track 209.2 -> 216.8 mm, vias 2 -> 7
- net FUNC: track 45.6 -> 40.2 mm, vias 4 -> 2
- net N$3: track 9.90 -> 13.6 mm
- net LED: track 3.01 -> 6.09 mm
- net HC: track 3.71 -> 6.05 mm
- net N$10: track 39.3 -> 38.8 mm
- net N$9: track 21.1 -> 20.6 mm

Commit message: rerouted some tracks
rerouted some tracks
Parts:
- moved R8 3.64 mm to (53.5, 19.9)
- moved D3 3.12 mm to (56.9, 28.2)
- moved R10 2.80 mm to (65.4, 12.9), turned to 180 degrees
- moved S2 2.62 mm to (74.3, 9.37)
- moved S1 2.25 mm to (65.8, 9.37)
- moved C3 1.88 mm to (40.0, 33.4)
- moved C5 1.13 mm to (41.0, 23.5)
- moved C2 1.12 mm to (38.9, 23.5)
- moved IC2 1.12 mm to (57.2, 14.5)
- moved SV3 0.91 mm to (71.9, 35.4)
- moved S3 0.75 mm to (32.1, 9.37)
- moved C10 0.40 mm to (39.9, 14.8)
- moved U$2 0.38 mm to (50.2, 14.0)
- moved C9 0.25 mm to (39.9, 12.5)
- moved Q1 0.25 mm to (40.9, 29.0)
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Connections:
- net +5V: no longer IC1.20
- net FUNC: now also IC1.23; no longer IC1.22
- net SCL: no longer R10.2
Routing:
- net GND: track 89.6 -> 123.1 mm, vias 6 -> 8
- net +5V: track 216.8 -> 196.3 mm, vias 7 -> 6
- net SCL: track 27.6 -> 18.4 mm
- net MINUTE: track 34.9 -> 39.1 mm
- net FUNC: track 40.2 -> 37.5 mm
- net LED: track 6.09 -> 3.92 mm
- net F: track 3.97 -> 5.30 mm
- net N$4: track 8.21 -> 6.98 mm
- net N$1: track 9.69 -> 10.8 mm
- net N$2: track 7.10 -> 8.13 mm
- net DP: track 6.49 -> 7.48 mm
- net D: track 4.08 -> 5.05 mm
- net HOUR: track 28.7 -> 29.5 mm
- net E: track 3.89 -> 4.76 mm
- net G: track 5.30 -> 6.08 mm
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Other:
- board size 70.8 x 29.5 mm -> 67.9 x 29.8 mm
- board text added: "FaberSpace"

Commit message: added final BOM
added final BOM
Parts:
- moved D1 1.46 mm to (31.5, 24.6), turned to 0 degrees
Routing:
- net GND: track 123.1 -> 103.7 mm, vias 8 -> 7
- net +5V: track 196.3 -> 186.9 mm
